Commit message: added simplified collision box

File: opr_description/urdf/version4/arms/left_arm.urdf.xacro (robot description, xacro)
@@ -36,4 +36,10 @@
       </geometry>
     </visual>
+    <collision>
+      <origin xyz="0.0 0.01763494312763214 -1.0798288327200158e-18" rpy="-3.141592653589793 1.5707963267948966 0.0"/>
+      <geometry>
+        <box size="0.03200000151991844 0.04626988619565964 0.0502999983727932"/>
+      </geometry>
+    </collision>
   </link>
   <link name="left_arm_link">
@@ -44,9 +50,14 @@
     </inertial>
     <visual>
-      <origin xyz="0 0 0" rpy="0 0 0"/>
       <geometry>
         <mesh filename="package://opr_description/meshes/version4/LeftUpperArm.stl"/>
       </geometry>
     </visual>
+    <collision>
+      <origin xyz="9.999983012676572e-05 9.999983012676239e-05 -0.05449999962002039" rpy="3.141592653589793 -0.0 1.5707963267948966"/>
+      <geometry>
+        <box size="0.045299999415874474 0.04529999941587448 0.132999999448657"/>
+      </geometry>
+    </collision>
   </link>
   <link name="left_forearm_link">
@@ -57,9 +68,14 @@
     </inertial>
     <visual>
-      <origin xyz="0 0 0" rpy="0 0 0"/>
       <geometry>
         <mesh filename="package://opr_description/meshes/version4/ForeArm.stl"/>
       </geometry>
     </visual>
+    <collision>
+      <origin xyz="1.6544247971531333e-34 2.7018807354169517e-18 -0.10078542958945036" rpy="3.141592653589793 -0.0 3.141592653589793"/>
+      <geometry>
+        <box size="0.02500000037252903 0.05029999837279319 0.2233708593994379"/>
+      </geometry>
+    </collision>
   </link>
 </robot>

File: opr_description/urdf/version4/arms/right_arm.urdf.xacro (robot description, xacro)
@@ -36,4 +36,10 @@
       </geometry>
     </visual>
+    <collision>
+      <origin xyz="0.0 -0.01763494312763214 -1.0798288327200158e-18" rpy="-7.498798913309288e-33 -1.5707963267948966 0.0"/>
+      <geometry>
+        <box size="0.03200000151991844 0.04626988619565964 0.0502999983727932"/>
+      </geometry>
+    </collision>
   </link>
   <link name="right_arm_link">
@@ -44,9 +50,14 @@
     </inertial>
     <visual>
-      <origin xyz="0 0 0" rpy="0 0 0"/>
       <geometry>
         <mesh filename="package://opr_description/meshes/version4/RightUpperArm.stl"/>
       </geometry>
     </visual>
+    <collision>
+      <origin xyz="-9.999983012675906e-05 9.999983012676239e-05 -0.05449999962002039" rpy="3.141592653589793 -0.0 1.5707963267948966"/>
+      <geometry>
+        <box size="0.045299999415874474 0.04529999941587448 0.132999999448657"/>
+      </geometry>
+    </collision>
   </link>
   <link name="right_forearm_link">
@@ -62,4 +73,10 @@
       </geometry>
     </visual>
+    <collision>
+      <origin xyz="-4.9632743914594e-34 -2.7018807354169517e-18 -0.10078542958945036" rpy="3.141592653589793 -0.0 -1.8369701987210297e-16"/>
+      <geometry>
+        <box size="0.02500000037252903 0.05029999837279319 0.2233708593994379"/>
+      </geometry>
+    </collision>
   </link>
 </robot>

File: opr_description/urdf/version4/body/body.urdf.xacro (robot description, xacro)
@@ -19,4 +19,10 @@
       </geometry>
     </visual>
+    <collision>
+      <origin xyz="-0.03270612440339107 -0.00010220211766156579 -0.007181904014356449" rpy="-2.882630121591322 -0.0013257236025648262 1.5704451281988223"/>
+      <geometry>
+        <box size="0.14548409358720668 0.1783637674020797 0.2041607213195921"/>
+      </geometry>
+    </collision>
   </link>
 </robot>

File: opr_description/urdf/version4/head/head.urdf.xacro (robot description, xacro)
@@ -21,4 +21,10 @@
       </geometry>
     </visual>
+    <collision>
+      <origin xyz="0.0045492063207171664 8.625779647839552e-19 0.049218710724377945" rpy="-3.141592653589793 0.5153769953275367 -1.2246467991473535e-16"/>
+      <geometry>
+        <box size="0.06765749574662422 0.07400000095367433 0.1137128056371003"/>
+      </geometry>
+    </collision>
   </link>
 </robot>

File: opr_description/urdf/version4/legs/left_leg.urdf.xacro (robot description, xacro)
@@ -99,4 +99,10 @@
       </geometry>
     </visual>
+    <collision>
+      <origin xyz="-0.00899999961256981 1.760429748682414e-18 -0.019749999977648258" rpy="-1.5707963267948966 6.123233995736766e-17 -1.5707963267948968"/>
+      <geometry>
+        <box size="0.03404976800084115 0.05949999950826168 0.06780000030994415"/>
+      </geometry>
+    </collision>
   </link>
   <link name="left_waist_roll_link">
@@ -111,4 +117,10 @@
       </geometry>
     </visual>
+    <collision>
+      <origin xyz="-0.009413216904900764 3.2907542331266094e-19 0.0040390074015276105" rpy="-1.5707963267948972 -1.4688870082426757 -3.1415926535897927"/>
+      <geometry>
+        <box size="0.05523091202205781 0.06322201062974908 0.06750000268220901"/>
+      </geometry>
+    </collision>
   </link>
   <link name="left_thigh_link">
@@ -123,4 +135,10 @@
       </geometry>
     </visual>
+    <collision>
+      <origin xyz="0.006775000132620336 0.0 -0.051994965644553304" rpy="0.0 6.123233995736766e-17 3.141592653589793"/>
+      <geometry>
+        <box size="0.0364500004798174 0.06949999928474425 0.11798530584201215"/>
+      </geometry>
+    </collision>
   </link>
   <link name="left_knee_link">
@@ -135,4 +153,10 @@
       </geometry>
     </visual>
+    <collision>
+      <origin xyz="-0.014478202443569897 0.0 -0.02849999815225601" rpy="0.0 6.123233995736766e-17 3.141592653589793"/>
+      <geometry>
+        <box size="0.05348143819719554 0.067500002682209 0.09397687017917632"/>
+      </geometry>
+    </collision>
   </link>
   <link name="left_shin_link">
@@ -147,4 +171,10 @@
       </geometry>
     </visual>
+    <collision>
+      <origin xyz="0.006775000132620334 0.0 -0.048005031887441874" rpy="0.0 6.123233995736766e-17 3.141592653589793"/>
+      <geometry>
+        <box size="0.03645000047981739 0.06949999928474429 0.11798530351370574"/>
+      </geometry>
+    </collision>
   </link>
   <link name="left_ankle_side_link">
@@ -159,4 +189,10 @@
       </geometry>
     </visual>
+    <collision>
+      <origin xyz="-0.011412393954674374 7.146761672779402e-20 0.01024523919989034" rpy="-1.5707963267948968 0.8390271244240705 3.141592653589793"/>
+      <geometry>
+        <box size="0.0249935555395753 0.055670833089966454 0.06750000268220901"/>
+      </geometry>
+    </collision>
   </link>
   <link name="left_ankle_link">
@@ -171,4 +207,10 @@
       </geometry>
     </visual>
+    <collision>
+      <origin xyz="-0.031873343670665126 9.999983012676639e-05 0.011302715725048419" rpy="1.4879617929266074 -1.0132707696249239e-17 -1.5707963267948968"/>
+      <geometry>
+        <box size="0.052299998700618744 0.053995914426129804 0.11384617313910501"/>
+      </geometry>
+    </collision>
   </link>
   <link name="left_foot_link">
@@ -183,4 +225,10 @@
       </geometry>
     </visual>
+    <collision>
+      <origin xyz="0.021000001579523087 0.020999998785555363 -0.023049999959766865" rpy="-3.141592653589793 1.5707963267948966 0.0"/>
+      <geometry>
+        <box size="0.0679000001400709 0.09249999932944773 0.17650000005960464"/>
+      </geometry>
+    </collision>
   </link>
   <link name="left_slider_crank_link">
@@ -195,4 +243,10 @@
       </geometry>
     </visual>
+    <collision>
+      <origin xyz="-0.0019685261027502948 -0.00014165545717062836 0.009035958319609934" rpy="0.016349194943953056 -0.2745921378361106 -0.0044335217605196925"/>
+      <geometry>
+        <box size="0.014016020056229879 0.02245286538792845 0.040529081872101635"/>
+      </geometry>
+    </collision>
   </link>
   <link name="left_hamstring_link">
@@ -207,4 +261,10 @@
       </geometry>
     </visual>
+    <collision>
+      <origin xyz="0.0026293317787349224 -1.6100013733620697e-19 -0.05002261372283101" rpy="3.141592653589793 -0.0 -6.123233995736766e-17"/>
+      <geometry>
+        <box size="0.022158662788569927 0.06949999928474428 0.11685264762490986"/>
+      </geometry>
+    </collision>
   </link>
   <link name="left_calf_link">
@@ -219,4 +279,10 @@
       </geometry>
     </visual>
+    <collision>
+      <origin xyz="0.0026293317787349224 -1.6100013733620697e-19 -0.049977388232946396" rpy="3.141592653589793 -0.0 -6.123233995736766e-17"/>
+      <geometry>
+        <box size="0.022158662788569927 0.06949999928474428 0.11685264855623244"/>
+      </geometry>
+    </collision>
   </link>
 </robot>

File: opr_description/urdf/version4/legs/right_leg.urdf.xacro (robot description, xacro)
@@ -99,4 +99,10 @@
       </geometry>
     </visual>
+    <collision>
+      <origin xyz="-0.00899999961256981 1.760429748682414e-18 -0.019749999977648258" rpy="-1.5707963267948966 6.123233995736766e-17 -1.5707963267948968"/>
+      <geometry>
+        <box size="0.03404976800084115 0.05949999950826168 0.06780000030994415"/>
+      </geometry>
+    </collision>
   </link>
   <link name="right_waist_roll_link">
@@ -111,4 +117,10 @@
       </geometry>
     </visual>
+    <collision>
+      <origin xyz="-0.009413216904900764 3.2907542331266094e-19 0.0040390074015276105" rpy="-1.5707963267948972 -1.4688870082426757 -3.1415926535897927"/>
+      <geometry>
+        <box size="0.05523091202205781 0.06322201062974908 0.06750000268220901"/>
+      </geometry>
+    </collision>
   </link>
   <link name="right_thigh_link">
@@ -123,4 +135,10 @@
       </geometry>
     </visual>
+    <collision>
+      <origin xyz="0.006775000132620336 0.0 -0.051994965644553304" rpy="0.0 6.123233995736766e-17 3.141592653589793"/>
+      <geometry>
+        <box size="0.0364500004798174 0.06949999928474425 0.11798530584201215"/>
+      </geometry>
+    </collision>
   </link>
   <link name="right_knee_link">
@@ -135,4 +153,10 @@
       </geometry>
     </visual>
+    <collision>
+      <origin xyz="-0.013864013366401194 0.0 -0.028499998152256012" rpy="0.0 6.123233995736766e-17 3.141592653589793"/>
+      <geometry>
+        <box size="0.05348143912851811 0.067500002682209 0.09397687017917632"/>
+      </geometry>
+    </collision>
   </link>
   <link name="right_shin_link">
@@ -147,4 +171,10 @@
       </geometry>
     </visual>
+    <collision>
+      <origin xyz="0.006775000132620334 0.0 -0.048005031887441874" rpy="0.0 6.123233995736766e-17 3.141592653589793"/>
+      <geometry>
+        <box size="0.03645000047981739 0.06949999928474429 0.11798530351370574"/>
+      </geometry>
+    </collision>
   </link>
   <link name="right_ankle_side_link">
@@ -159,4 +189,10 @@
       </geometry>
     </visual>
+    <collision>
+      <origin xyz="-0.011412393954674374 7.146761672779402e-20 0.01024523919989034" rpy="-1.5707963267948968 0.8390271244240705 3.141592653589793"/>
+      <geometry>
+        <box size="0.0249935555395753 0.055670833089966454 0.06750000268220901"/>
+      </geometry>
+    </collision>
   </link>
   <link name="right_ankle_link">
@@ -171,4 +207,10 @@
       </geometry>
     </visual>
+    <collision>
+      <origin xyz="-0.031873343670665126 9.999983012676639e-05 0.011302715725048419" rpy="1.4879617929266074 -1.0132707696249239e-17 -1.5707963267948968"/>
+      <geometry>
+        <box size="0.052299998700618744 0.053995914426129804 0.11384617313910501"/>
+      </geometry>
+    </collision>
   </link>
   <link name="right_foot_link">
@@ -183,4 +225,10 @@
       </geometry>
     </visual>
+    <collision>
+      <origin xyz="0.021000001579523087 -0.020999998785555363 -0.023049999959766865" rpy="-3.141592653589793 1.5707963267948966 0.0"/>
+      <geometry>
+        <box size="0.0679000001400709 0.09249999932944773 0.17650000005960464"/>
+      </geometry>
+    </collision>
   </link>
   <link name="right_slider_crank_link">
@@ -195,4 +243,10 @@
       </geometry>
     </visual>
+    <collision>
+      <origin xyz="-0.0019685261027502948 -0.00014165545717062836 0.009035958319609934" rpy="0.016349194943953056 -0.2745921378361106 -0.0044335217605196925"/>
+      <geometry>
+        <box size="0.014016020056229879 0.02245286538792845 0.040529081872101635"/>
+      </geometry>
+    </collision>
   </link>
   <link name="right_hamstring_link">
@@ -207,4 +261,10 @@
       </geometry>
     </visual>
+    <collision>
+      <origin xyz="0.0026293317787349224 -1.6100013733620697e-19 -0.05002261372283101" rpy="3.141592653589793 -0.0 -6.123233995736766e-17"/>
+      <geometry>
+        <box size="0.022158662788569927 0.06949999928474428 0.11685264762490986"/>
+      </geometry>
+    </collision>
   </link>
   <link name="right_calf_link">
@@ -219,4 +279,10 @@
       </geometry>
     </visual>
+    <collision>
+      <origin xyz="0.0026293317787349224 -1.6100013733620697e-19 -0.049977388232946396" rpy="3.141592653589793 -0.0 -6.123233995736766e-17"/>
+      <geometry>
+        <box size="0.022158662788569927 0.06949999928474428 0.11685264855623244"/>
+      </geometry>
+    </collision>
   </link>
 </robot>

Commit message: lighter mesh

File: opr_description/urdf/version4/arms/left_arm.urdf.xacro (robot description, xacro)
@@ -33,5 +33,5 @@
       <origin xyz="0 0 0" rpy="${PI/2} 0 0"/>
       <geometry>
-        <mesh filename="package://opr_description/meshes/version4/Shoulder.stl"/>
+        <mesh filename="package://opr_description/meshes/version4/ShoulderLight.stl"/>
       </geometry>
     </visual>
@@ -47,9 +47,9 @@
       <origin xyz="-0.000173 -0.000173 -0.0545" rpy="0 0 0"/>
       <mass value="0.198342"/>
-        <inertia ixx="0.000398226787" ixy="0.000000017648" ixz="-0.000003440285" iyy="0.000398226787" iyz="0.000003440285" izz="0.000042097457"/>
+      <inertia ixx="0.000398226787" ixy="0.000000017648" ixz="-0.000003440285" iyy="0.000398226787" iyz="0.000003440285" izz="0.000042097457"/>
     </inertial>
     <visual>
       <geometry>
-        <mesh filename="package://opr_description/meshes/version4/LeftUpperArm.stl"/>
+        <mesh filename="package://opr_description/meshes/version4/LeftUpperArmLight.stl"/>
       </geometry>
     </visual>
@@ -69,5 +69,5 @@
     <visual>
       <geometry>
-        <mesh filename="package://opr_description/meshes/version4/ForeArm.stl"/>
+        <mesh filename="package://opr_description/meshes/version4/ForeArmLight.stl"/>
       </geometry>
     </visual>

File: opr_description/urdf/version4/arms/right_arm.urdf.xacro (robot description, xacro)
@@ -33,5 +33,5 @@
       <origin xyz="0 0 0" rpy="${-PI/2} 0 0"/>
       <geometry>
-        <mesh filename="package://opr_description/meshes/version4/Shoulder.stl"/>
+        <mesh filename="package://opr_description/meshes/version4/ShoulderLight.stl"/>
       </geometry>
     </visual>
@@ -51,5 +51,5 @@
     <visual>
       <geometry>
-        <mesh filename="package://opr_description/meshes/version4/RightUpperArm.stl"/>
+        <mesh filename="package://opr_description/meshes/version4/RightUpperArmLight.stl"/>
       </geometry>
     </visual>
@@ -70,5 +70,5 @@
       <origin xyz="0 0 0" rpy="0 0 ${PI}"/>
       <geometry>
-        <mesh filename="package://opr_description/meshes/version4/ForeArm.stl"/>
+        <mesh filename="package://opr_description/meshes/version4/ForeArmLight.stl"/>
       </geometry>
     </visual>

File: opr_description/urdf/version4/body/body.urdf.xacro (robot description, xacro)
@@ -16,5 +16,5 @@
     <visual>
       <geometry>
-        <mesh filename="package://opr_description/meshes/version4/Trunk.stl"/>
+        <mesh filename="package://opr_description/meshes/version4/TrunkLight.stl"/>
       </geometry>
     </visual>

File: opr_description/urdf/version4/head/head.urdf.xacro (robot description, xacro)
@@ -18,5 +18,5 @@
     <visual>
       <geometry>
-        <mesh filename="package://opr_description/meshes/version4/Head.stl"/>
+        <mesh filename="package://opr_description/meshes/version4/HeadLight.stl"/>
       </geometry>
     </visual>

File: opr_description/urdf/version4/legs/left_leg.urdf.xacro (robot description, xacro)
@@ -96,5 +96,5 @@
     <visual>
       <geometry>
-        <mesh filename="package://opr_description/meshes/version4/WaistYaw.stl"/>
+        <mesh filename="package://opr_description/meshes/version4/WaistYawLight.stl"/>
       </geometry>
     </visual>
@@ -114,5 +114,5 @@
     <visual>
       <geometry>
-        <mesh filename="package://opr_description/meshes/version4/WaistRoll.stl"/>
+        <mesh filename="package://opr_description/meshes/version4/WaistRollLight.stl"/>
       </geometry>
     </visual>
@@ -132,5 +132,5 @@
     <visual>
       <geometry>
-        <mesh filename="package://opr_description/meshes/version4/Thigh.stl"/>
+        <mesh filename="package://opr_description/meshes/version4/ThighLight.stl"/>
       </geometry>
     </visual>
@@ -150,5 +150,5 @@
     <visual>
       <geometry>
-        <mesh filename="package://opr_description/meshes/version4/LeftKnee.stl"/>
+        <mesh filename="package://opr_description/meshes/version4/LeftKneeLight.stl"/>
       </geometry>
     </visual>
@@ -168,5 +168,5 @@
     <visual>
       <geometry>
-        <mesh filename="package://opr_description/meshes/version4/Shin.stl"/>
+        <mesh filename="package://opr_description/meshes/version4/ShinLight.stl"/>
       </geometry>
     </visual>
@@ -186,5 +186,5 @@
     <visual>
       <geometry>
-        <mesh filename="package://opr_description/meshes/version4/AnkleSide.stl"/>
+        <mesh filename="package://opr_description/meshes/version4/AnkleSideLight.stl"/>
       </geometry>
     </visual>
@@ -204,5 +204,5 @@
     <visual>
       <geometry>
-        <mesh filename="package://opr_description/meshes/version4/Ankle.stl"/>
+        <mesh filename="package://opr_description/meshes/version4/AnkleLight.stl"/>
       </geometry>
     </visual>
@@ -222,5 +222,5 @@
     <visual>
       <geometry>
-        <mesh filename="package://opr_description/meshes/version4/LeftFoot.stl"/>
+        <mesh filename="package://opr_description/meshes/version4/LeftFootLight.stl"/>
       </geometry>
     </visual>
@@ -236,9 +236,9 @@
       <origin xyz="-0.002952 0 0.01162" rpy="0 0 0"/>
       <mass value="0.008594"/>
-    <inertia ixx="0.000000938108" ixy="0" ixz="-0.000000173459" iyy="0.000000887351" iyz="-0.000000000002" izz="0.000000292478"/>
-    </inertial>
-    <visual>
-      <geometry>
-        <mesh filename="package://opr_description/meshes/version4/SliderCrank.stl"/>
+      <inertia ixx="0.000000938108" ixy="0" ixz="-0.000000173459" iyy="0.000000887351" iyz="-0.000000000002" izz="0.000000292478"/>
+    </inertial>
+    <visual>
+      <geometry>
+        <mesh filename="package://opr_description/meshes/version4/SliderCrankLight.stl"/>
       </geometry>
     </visual>
@@ -258,5 +258,5 @@
     <visual>
       <geometry>
-        <mesh filename="package://opr_description/meshes/version4/Hamstring.stl"/>
+        <mesh filename="package://opr_description/meshes/version4/HamstringLight.stl"/>
       </geometry>
     </visual>
@@ -276,5 +276,5 @@
     <visual>
       <geometry>
-        <mesh filename="package://opr_description/meshes/version4/Calf.stl"/>
+        <mesh filename="package://opr_description/meshes/version4/CalfLight.stl"/>
       </geometry>
     </visual>

File: opr_description/urdf/version4/legs/right_leg.urdf.xacro (robot description, xacro)
@@ -96,5 +96,5 @@
     <visual>
       <geometry>
-        <mesh filename="package://opr_description/meshes/version4/WaistYaw.stl"/>
+        <mesh filename="package://opr_description/meshes/version4/WaistYawLight.stl"/>
       </geometry>
     </visual>
@@ -114,5 +114,5 @@
     <visual>
       <geometry>
-        <mesh filename="package://opr_description/meshes/version4/WaistRoll.stl"/>
+        <mesh filename="package://opr_description/meshes/version4/WaistRollLight.stl"/>
       </geometry>
     </visual>
@@ -132,5 +132,5 @@
     <visual>
       <geometry>
-        <mesh filename="package://opr_description/meshes/version4/Thigh.stl"/>
+        <mesh filename="package://opr_description/meshes/version4/ThighLight.stl"/>
       </geometry>
     </visual>
@@ -150,5 +150,5 @@
     <visual>
       <geometry>
-        <mesh filename="package://opr_description/meshes/version4/RightKnee.stl"/>
+        <mesh filename="package://opr_description/meshes/version4/RightKneeLight.stl"/>
       </geometry>
     </visual>
@@ -168,5 +168,5 @@
     <visual>
       <geometry>
-        <mesh filename="package://opr_description/meshes/version4/Shin.stl"/>
+        <mesh filename="package://opr_description/meshes/version4/ShinLight.stl"/>
       </geometry>
     </visual>
@@ -186,5 +186,5 @@
     <visual>
       <geometry>
-        <mesh filename="package://opr_description/meshes/version4/AnkleSide.stl"/>
+        <mesh filename="package://opr_description/meshes/version4/AnkleSideLight.stl"/>
       </geometry>
     </visual>
@@ -204,5 +204,5 @@
     <visual>
       <geometry>
-        <mesh filename="package://opr_description/meshes/version4/Ankle.stl"/>
+        <mesh filename="package://opr_description/meshes/version4/AnkleLight.stl"/>
       </geometry>
     </visual>
@@ -222,5 +222,5 @@
     <visual>
       <geometry>
-        <mesh filename="package://opr_description/meshes/version4/RightFoot.stl"/>
+        <mesh filename="package://opr_description/meshes/version4/RightFootLight.stl"/>
       </geometry>
     </visual>
@@ -236,9 +236,9 @@
       <origin xyz="-0.002952 0 0.01162" rpy="0 0 0"/>
       <mass value="0.008594"/>
-    <inertia ixx="0.000000938108" ixy="0" ixz="-0.000000173459" iyy="0.000000887351" iyz="-0.000000000002" izz="0.000000292478"/>
-    </inertial>
-    <visual>
-      <geometry>
-        <mesh filename="package://opr_description/meshes/version4/SliderCrank.stl"/>
+      <inertia ixx="0.000000938108" ixy="0" ixz="-0.000000173459" iyy="0.000000887351" iyz="-0.000000000002" izz="0.000000292478"/>
+    </inertial>
+    <visual>
+      <geometry>
+        <mesh filename="package://opr_description/meshes/version4/SliderCrankLight.stl"/>
       </geometry>
     </visual>
@@ -258,5 +258,5 @@
     <visual>
       <geometry>
-        <mesh filename="package://opr_description/meshes/version4/Hamstring.stl"/>
+        <mesh filename="package://opr_description/meshes/version4/HamstringLight.stl"/>
       </geometry>
     </visual>
@@ -276,5 +276,5 @@
     <visual>
       <geometry>
-        <mesh filename="package://opr_description/meshes/version4/Calf.stl"/>
+        <mesh filename="package://opr_description/meshes/version4/CalfLight.stl"/>
       </geometry>
     </visual>
