Commit message: fix inertial

File: opr_description/robots/gankenkun_v4.xacro (robot description, xacro)
@@ -1,5 +1,6 @@
 <?xml version="1.0"?>
 <robot xmlns:xacro="http://www.ros.org/wiki/xacro" name="gankenkun">
-  <!--Constants for robot dimensions -->
+  <!--Constants
+  for robot dimensions -->
   <xacro:property name="PI" value="3.1415926535897931"/>
   <!-- Import Rviz color -->
@@ -8,12 +9,10 @@
   <link name="base_link"/>
   <!-- uncomment this part to fixed the body in space (ignore gravity) -->
-  <!--
-  <link name="world"/>
+  <!-- <link name="world"/>
   <joint name="world2base" type="fixed">
-    <origin xyz="0 0 0" rpy="0 0 0" />
+    <origin xyz="0 0 0" rpy="0 0 0"/>
     <parent link="world"/>
     <child link="base_link"/>
-  </joint>
-  -->
+  </joint> -->
   <!-- import robot parts -->
   <xacro:include filename="$(find opr_description)/urdf/version4/body/body.urdf.xacro"/>
@@ -25,4 +24,5 @@
   <!-- gazebo reference -->
   <xacro:include filename="$(find opr_description)/urdf/gazebo.xacro"/>
+  <xacro:include filename="$(find opr_description)/urdf/version4/body/body.gazebo.xacro"/>
   <xacro:include filename="$(find opr_description)/urdf/version4/head/head.gazebo.xacro"/>
   <xacro:include filename="$(find opr_description)/urdf/version4/arms/arms.gazebo.xacro"/>

File: opr_description/urdf/version4/arms/arms.gazebo.xacro (robot description, xacro)
@@ -5,5 +5,5 @@
       <mu1>1.0</mu1>
       <mu2>1.0</mu2>
-      <kp>10000.0</kp>
+      <kp>1000000.0</kp>
       <kd>100.0</kd>
       <gravity>false</gravity>

File: opr_description/urdf/version4/arms/arms.transmission.xacro (robot description, xacro)
@@ -13,8 +13,8 @@
   </xacro:macro>
   <xacro:arm_transmission name="left_shoulder_pitch_joint"/>
-  <xacro:arm_transmission name="left_shoulder_roll_joint"/>
+  <!-- <xacro:arm_transmission name="left_shoulder_roll_joint"/> -->
   <xacro:arm_transmission name="left_elbow_pitch_joint"/>
   <xacro:arm_transmission name="right_shoulder_pitch_joint"/>
-  <xacro:arm_transmission name="right_shoulder_roll_joint"/>
+  <!-- <xacro:arm_transmission name="right_shoulder_roll_joint"/> -->
   <xacro:arm_transmission name="right_elbow_pitch_joint"/>
 </robot>

File: opr_description/urdf/version4/arms/left_arm.urdf.xacro (robot description, xacro)
@@ -6,5 +6,5 @@
     <child link="left_shoulder_link"/>
     <origin xyz="0 0.0615 0.056" rpy="0 0 0"/>
-    <limit effort="100" lower="${-3*PI/4}" upper="${3*PI/4}" velocity="4.8"/>
+    <limit effort="1000" lower="${-3*PI/4}" upper="${3*PI/4}" velocity="4.8"/>
     <axis xyz="0 1 0"/>
   </joint>
@@ -26,7 +26,7 @@
   <link name="left_shoulder_link">
     <inertial>
-      <origin xyz="0 0 -0.007843" rpy="${PI/2} 0 0"/>
+      <origin xyz="0 0.007843 0" rpy="${PI/2} 0 0"/>
       <mass value="0.031036"/>
-      <inertia ixx="0.006857020" ixy="0" iyy="0.012483012" ixz="0" iyz="0" izz="0.014531649"/>
+      <inertia ixx="0.000006857020" ixy="0.0" ixz="0.0" izz="0.000012483012" iyz="0.0" iyy="0.000014531649"/>
     </inertial>
     <visual>
@@ -47,5 +47,5 @@
       <origin xyz="-0.000173 -0.000173 -0.0545" rpy="0 0 0"/>
       <mass value="0.198342"/>
-      <inertia ixx="0.000398226787" ixy="0.000017648" ixz="-0.0003440285" iyy="0.000398226787" iyz="0.0003440285" izz="0.00042097457"/>
+        <inertia ixx="0.000398226787" ixy="0.000000017648" ixz="-0.000003440285" iyy="0.000398226787" iyz="0.000003440285" izz="0.000042097457"/>
     </inertial>
     <visual>
@@ -63,7 +63,7 @@
   <link name="left_forearm_link">
     <inertial>
-      <origin xyz="0 0.009824 -0.126417" rpy="-0.095493 0 0"/>
+      <origin xyz="0 0.009824 -0.126417" rpy="0 0 0"/>
       <mass value="0.06313"/>
-      <inertia ixx="0.000296886941" ixy="0" ixz="0" iyy="0.000284555999" iyz="0" izz="0.000016240155"/>
+      <inertia ixx="0.000296886941" ixy="0.000000000007" ixz="-0.000000000026" iyy="0.000284555999" iyz="-0.000025954170" izz="0.000016240155"/>
     </inertial>
     <visual>

File: opr_description/urdf/version4/arms/right_arm.urdf.xacro (robot description, xacro)
@@ -6,5 +6,5 @@
     <child link="right_shoulder_link"/>
     <origin xyz="0 -0.0615 0.056" rpy="0 0 0"/>
-    <limit effort="100" lower="${-3*PI/4}" upper="${3*PI/4}" velocity="4.8"/>
+    <limit effort="1000" lower="${-3*PI/4}" upper="${3*PI/4}" velocity="4.8"/>
     <axis xyz="0 1 0"/>
   </joint>
@@ -26,7 +26,7 @@
   <link name="right_shoulder_link">
     <inertial>
-      <origin xyz="0 0 -0.007843" rpy="${-PI/2} 0 0"/>
+      <origin xyz="0 -0.007843 0" rpy="${-PI/2} 0 0"/>
       <mass value="0.031036"/>
-      <inertia ixx="0.006857020" ixy="0" iyy="0.012483012" ixz="0" iyz="0" izz="0.014531649"/>
+      <inertia ixx="0.000006857020" ixy="0.0" ixz="0.0" izz="0.000012483012" iyz="0.0" iyy="0.000014531649"/>
     </inertial>
     <visual>
@@ -45,7 +45,7 @@
   <link name="right_arm_link">
     <inertial>
-      <origin xyz="0.00049 -0.00049 -0.0545" rpy="0.000873 -0.000873 -0.785398"/>
+      <origin xyz="0.00049 -0.00049 -0.0545" rpy="0 0 0"/>
       <mass value="0.198342"/>
-      <inertia ixx="0.00398185104" ixy="0.00000071266" ixz="0.00000295835" iyy="0.00398185104" iyz="0.00000295835" izz="0.00042014091"/>
+      <inertia ixx="0.000398185104" ixy="0.000000071266" ixz="0.000000295835" iyy="0.000398185104" iyz="0.000000295835" izz="0.000042014091"/>
     </inertial>
     <visual>
@@ -63,7 +63,7 @@
   <link name="right_forearm_link">
     <inertial>
-      <origin xyz="0 0.009824 -0.126417" rpy="-0.095493 0 ${PI}"/>
+      <origin xyz="0 -0.009824 -0.126417" rpy="0 0 ${PI}"/>
       <mass value="0.06313"/>
-      <inertia ixx="0.000296886941" ixy="0" ixz="0" iyy="0.000284555999" iyz="0" izz="0.000016240155"/>
+      <inertia ixx="0.000296886941" ixy="0.000000000007" ixz="-0.000000000026" iyy="0.000284555999" iyz="-0.000025954170" izz="0.000016240155"/>
     </inertial>
     <visual>

File: opr_description/urdf/version4/body/body.urdf.xacro (robot description, xacro)
@@ -10,7 +10,7 @@
   <link name="body_link">
     <inertial>
-      <origin xyz="-0.022825 0.000073 -0.01572" rpy="0.001047 0.110657 0.022516"/>
+      <origin xyz="-0.022825 0.000073 -0.015720" rpy="0 0 0"/>
       <mass value="1.645331"/>
-      <inertia ixx="7.742297482" ixy="-0.005961013" ixz="-0.422502364" iyy="8.034384246" iyz="0.003797186" izz="3.984603997"/>
+      <inertia ixx="0.007742297482" ixy="0.000005961013" ixz="0.000422502364" iyy="0.008034384246" iyz="-0.000003797186" izz="0.003984603997"/>
     </inertial>
     <visual>

File: opr_description/urdf/version4/head/head.urdf.xacro (robot description, xacro)
@@ -12,7 +12,7 @@
   <link name="head_yaw_link">
     <inertial>
-      <origin xyz="0.019189 -0.000533 0.057803" rpy="0.00523598 -0.719842 0.00436332"/>
+      <origin xyz="0.019189 -0.000533 0.057803" rpy="0 0 0"/>
       <mass value="0.160477"/>
-      <inertia ixx="0.135811588" ixy="0.293359" iyy="0.151374671" ixz="0.41997404" iyz="0.078967" izz="0.124729778"/>
+      <inertia ixx="0.000135811588" ixy="-0.000000293359" ixz="-0.000041997404" iyy="0.000151374671" iyz="-0.000000078967" izz="0.000124729778"/>
     </inertial>
     <visual>

File: opr_description/urdf/version4/legs/left_leg.urdf.xacro (robot description, xacro)
@@ -90,7 +90,7 @@
   <link name="left_waist_yaw_link">
     <inertial>
-      <origin xyz="0.008607 -0.000 0.008006" rpy="0 0.00087 0"/>
+      <origin xyz="-0.008607 0 -0.008006" rpy="0 0 0"/>
       <mass value="0.038113"/>
-      <inertia ixx="0.00012431119" ixy="0" ixz="0.000000009667" iyy="0.00030968751" iyz="0" izz="0.00022812922"/>
+      <inertia ixx="0.000012431119" ixy="0" ixz="-0.000000009667" iyy="0.000030968751" iyz="0" izz="0.000022812922"/>
     </inertial>
     <visual>
@@ -108,7 +108,7 @@
   <link name="left_waist_roll_link">
     <inertial>
-      <origin xyz="-0.009956 0.000 0.002314" rpy="0 0 0"/>
+      <origin xyz="-0.009956 0 0.002314" rpy="0 0 0"/>
       <mass value="0.169734"/>
-      <inertia ixx="0.000063728705" ixy="0.0" ixz="0.0" iyy="0.000073380568" iyz="0.0" izz="0.000071098616"/>
+      <inertia ixx="0.000063728596" ixy="0" ixz="0.000008352459" iyy="0.000073380568" iyz="-0.000000058" izz="0.000071098724"/>
     </inertial>
     <visual>
@@ -126,5 +126,5 @@
   <link name="left_thigh_link">
     <inertial>
-      <origin xyz="0.011263 0.0 -0.054265" rpy="-0.317307 0.016236 -0.005585"/>
+      <origin xyz="0.011263 0 -0.054265" rpy="0 0 0"/>
       <mass value="0.042298"/>
       <inertia ixx="0.000070306" ixy="0" ixz="0" iyy="0.000040631" iyz="0" izz="0.000039265"/>
@@ -146,5 +146,5 @@
       <origin xyz="-0.013195 -0.000597 -0.028501" rpy="0 0 0"/>
       <mass value="0.292217"/>
-      <inertia ixx="0.309351160" ixy="0.002710035" ixz="-0.000001274" iyy="0.297482099" iyz="-0.000000102" izz="0.128014307"/>
+      <inertia ixx="0.000309351160" ixy="0.000002710035" ixz="-0.000000001274" iyy="0.000297482099" iyz="-0.000000000102" izz="0.000128014307"/>
     </inertial>
     <visual>
@@ -162,7 +162,7 @@
   <link name="left_shin_link">
     <inertial>
-      <origin xyz="0.011263 0.000000 0.045735" rpy="0 0 0"/>
+      <origin xyz="0.011263 0 -0.045735" rpy="0 0 0"/>
       <mass value="0.042298"/>
-      <inertia ixx="0.000070306" ixy="0" ixz="0.000000534" iyy="0.000040631" iyz="0.000000507" izz="0.000039265"/>
+      <inertia ixx="0.000070306" ixy="0" ixz="0" iyy="0.000040631" iyz="0" izz="0.000039265"/>
     </inertial>
     <visual>
@@ -180,5 +180,5 @@
   <link name="left_ankle_side_link">
     <inertial>
-      <origin xyz="-0.013347 0.0 0.008343" rpy="0 0 0"/>
+      <origin xyz="-0.013347 0 0.008343" rpy="0 0 0"/>
       <mass value="0.023147"/>
       <inertia ixx="0.000020167808" ixy="-0.000000045124" ixz="0.000002791677" iyy="0.000007373394" iyz="-0.000000072190" izz="0.000022888907"/>
@@ -198,7 +198,7 @@
   <link name="left_ankle_link">
     <inertial>
-      <origin xyz="-0.032373 -0.000347 0.005993" rpy="-0.05933 -0.16006 0.01135"/>
+      <origin xyz="-0.032373 0 0.005993" rpy="0 0 0"/>
       <mass value="0.251442"/>
-      <inertia ixx="0.00076837" ixy="0.00000308474" ixz="0.00033997201" iyy="0.002787734" iyz="0.000005228" izz="0.00281200733"/>
+      <inertia ixx="0.000076837363" ixy="-0.000000308474" ixz="-0.000033997201" iyy="0.000278773400" iyz="0" izz="0.000281200733"/>
     </inertial>
     <visual>
@@ -216,7 +216,7 @@
   <link name="left_foot_link">
     <inertial>
-      <origin xyz="0.020826 0.016517 -0.039217" rpy="0.096859 -0.022861 -0.038397"/>
+      <origin xyz="0.020826 0.016517 -0.039217" rpy="0 0 0"/>
       <mass value="0.098589"/>
-      <inertia ixx="0.00107804945" ixy="0.00009010661" ixz="-0.00008516149" iyy="0.00362837937" iyz="-0.00007813284" izz="0.00440229333"/>
+      <inertia ixx="0.000107804945" ixy="0.000009010661" ixz="-0.000008516149" iyy="0.000362837937" iyz="-0.000007813284" izz="0.000440229333"/>
     </inertial>
     <visual>
@@ -234,7 +234,7 @@
   <link name="left_slider_crank_link">
     <inertial>
-      <origin xyz="-0.002952 0.00009 0.011619" rpy="0.00767944 0.246632 0"/>
+      <origin xyz="-0.002952 0 0.01162" rpy="0 0 0"/>
       <mass value="0.008594"/>
-      <inertia ixx="0.000000938108" ixy="0" ixz="0" iyy="0.000000887315" iyz="0" izz="0.000000292514"/>
+    <inertia ixx="0.000000938108" ixy="0" ixz="-0.000000173459" iyy="0.000000887351" iyz="-0.000000000002" izz="0.000000292478"/>
     </inertial>
     <visual>
@@ -252,7 +252,7 @@
   <link name="left_hamstring_link">
     <inertial>
-      <origin xyz="-0.001824 0.000000 -0.047726" rpy="0 0 0"/>
+      <origin xyz="-0.001824 0 -0.047726" rpy="0 0 0"/>
       <mass value="0.029252"/>
-      <inertia ixx="0.000049199" ixy="0.000000" ixz="-0.000000651" iyy="0.000026577" iyz="-0.000000219" izz="0.000023937"/>
+      <inertia ixx="0.000049199945" ixy="0" ixz="-0.000000651855" iyy="0.000026577036" iyz="0" izz="0.00002393766"/>
     </inertial>
     <visual>
@@ -270,7 +270,7 @@
   <link name="left_calf_link">
     <inertial>
-      <origin xyz="-0.001824 0.000 -0.052274" rpy="0 0 0"/>
+      <origin xyz="-0.001824 0 -0.052274" rpy="0 0 0"/>
       <mass value="0.029252"/>
-      <inertia ixx="0.000049199945" ixy="0.000" ixz="0.000000651855" iyy="0.000026577036" iyz="-0.000000219226" izz="0.000023937660"/>
+      <inertia ixx="0.000049199945" ixy="0" ixz="0.000000651855" iyy="0.000026577036" iyz="0" izz="0.000023937660"/>
     </inertial>
     <visual>

File: opr_description/urdf/version4/legs/right_leg.urdf.xacro (robot description, xacro)
@@ -90,7 +90,7 @@
   <link name="right_waist_yaw_link">
     <inertial>
-      <origin xyz="0.008607 -0.000 0.008006" rpy="0 0.00087 0"/>
+      <origin xyz="-0.008607 0 -0.008006" rpy="0 0 0"/>
       <mass value="0.038113"/>
-      <inertia ixx="0.00012431119" ixy="0" ixz="0.000000009667" iyy="0.00030968751" iyz="0" izz="0.00022812922"/>
+      <inertia ixx="0.000012431119" ixy="0" ixz="-0.000000009667" iyy="0.000030968751" iyz="0" izz="0.000022812922"/>
     </inertial>
     <visual>
@@ -108,7 +108,7 @@
   <link name="right_waist_roll_link">
     <inertial>
-      <origin xyz="-0.009956 0.000 0.002314" rpy="0 0 0"/>
+      <origin xyz="-0.009956 0 0.002314" rpy="0 0 0"/>
       <mass value="0.169734"/>
-      <inertia ixx="0.000063728705" ixy="0.0" ixz="0.0" iyy="0.000073380568" iyz="0.0" izz="0.000071098616"/>
+      <inertia ixx="0.000063728596" ixy="0" ixz="0.000008352459" iyy="0.000073380568" iyz="-0.000000058" izz="0.000071098724"/>
     </inertial>
     <visual>
@@ -126,5 +126,5 @@
   <link name="right_thigh_link">
     <inertial>
-      <origin xyz="0.011263 0.0 -0.054265" rpy="-0.317307 0.016236 -0.005585"/>
+      <origin xyz="0.011263 0 -0.054265" rpy="0 0 0"/>
       <mass value="0.042298"/>
       <inertia ixx="0.000070306" ixy="0" ixz="0" iyy="0.000040631" iyz="0" izz="0.000039265"/>
@@ -144,7 +144,7 @@
   <link name="right_knee_link">
     <inertial>
-      <origin xyz="-0.013195 0.000597 -0.028499" rpy="0 0 0"/>
+      <origin xyz="-0.013195 0.000597 -0.028501" rpy="0 0 0"/>
       <mass value="0.292217"/>
-      <inertia ixx="0.00030935116" ixy="0" ixz="0" iyy="0.000297482099" iyz="0" izz="0.000128014307"/>
+      <inertia ixx="0.000309351160" ixy="-0.000002710035" ixz="0.000000001274" iyy="0.000297482099" iyz="-0.000000000102" izz="0.000128014307"/>
     </inertial>
     <visual>
@@ -162,7 +162,7 @@
   <link name="right_shin_link">
     <inertial>
-      <origin xyz="0.011263 0.000000 0.045735" rpy="0 0 0"/>
+      <origin xyz="0.011263 0 -0.045735" rpy="0 0 0"/>
       <mass value="0.042298"/>
-      <inertia ixx="0.000070306" ixy="0" ixz="0.000000534" iyy="0.000040631" iyz="0.000000507" izz="0.000039265"/>
+      <inertia ixx="0.000070306" ixy="0" ixz="0" iyy="0.000040631" iyz="0" izz="0.000039265"/>
     </inertial>
     <visual>
@@ -180,5 +180,5 @@
   <link name="right_ankle_side_link">
     <inertial>
-      <origin xyz="-0.013347 0.0 0.008343" rpy="0 0 0"/>
+      <origin xyz="-0.013347 0 0.008343" rpy="0 0 0"/>
       <mass value="0.023147"/>
       <inertia ixx="0.000020167808" ixy="-0.000000045124" ixz="0.000002791677" iyy="0.000007373394" iyz="-0.000000072190" izz="0.000022888907"/>
@@ -198,7 +198,7 @@
   <link name="right_ankle_link">
     <inertial>
-      <origin xyz="-0.032373 -0.000347 0.005993" rpy="-0.05933 -0.16006 0.01135"/>
+      <origin xyz="-0.032373 0 0.005993" rpy="0 0 0"/>
       <mass value="0.251442"/>
-      <inertia ixx="0.00076837" ixy="0.00000308474" ixz="0.00033997201" iyy="0.002787734" iyz="0.000005228" izz="0.00281200733"/>
+      <inertia ixx="0.000076837363" ixy="-0.000000308474" ixz="-0.000033997201" iyy="0.000278773400" iyz="0" izz="0.000281200733"/>
     </inertial>
     <visual>
@@ -216,7 +216,7 @@
   <link name="right_foot_link">
     <inertial>
-      <origin xyz="0.020826 -0.016517 -0.039217" rpy="-0.0968139 -0.022869 0.0383972"/>
+      <origin xyz="0.020826 -0.016517 -0.039217" rpy="0 0 0"/>
       <mass value="0.098589"/>
-      <inertia ixx="0.000107805" ixy="-0.000009011" ixz="-0.000008516" iyy="0.000362838" iyz="0.000007813" izz="0.000440229"/>
+      <inertia ixx="0.000107804945" ixy="-0.000009010661" ixz="-0.000008516149" iyy="0.000362837937" iyz="0.000007813284" izz="0.000440229333"/>
     </inertial>
     <visual>
@@ -234,7 +234,7 @@
   <link name="right_slider_crank_link">
     <inertial>
-      <origin xyz="-0.002952 0.00009 0.011619" rpy="0.00767944 0.246632 0"/>
+      <origin xyz="-0.002952 0 0.01162" rpy="0 0 0"/>
       <mass value="0.008594"/>
-      <inertia ixx="0.000000938108" ixy="0" ixz="0" iyy="0.000000887315" iyz="0" izz="0.000000292514"/>
+    <inertia ixx="0.000000938108" ixy="0" ixz="-0.000000173459" iyy="0.000000887351" iyz="-0.000000000002" izz="0.000000292478"/>
     </inertial>
     <visual>
@@ -252,7 +252,7 @@
   <link name="right_hamstring_link">
     <inertial>
-      <origin xyz="-0.001824 0.000000 -0.047726" rpy="0 0 0"/>
+      <origin xyz="-0.001824 0 -0.047726" rpy="0 0 0"/>
       <mass value="0.029252"/>
-      <inertia ixx="0.000049199" ixy="0.000000" ixz="-0.000000651" iyy="0.000026577" iyz="-0.000000219" izz="0.000023937"/>
+      <inertia ixx="0.000049199945" ixy="0" ixz="-0.000000651855" iyy="0.000026577036" iyz="0" izz="0.00002393766"/>
     </inertial>
     <visual>
@@ -270,7 +270,7 @@
   <link name="right_calf_link">
     <inertial>
-      <origin xyz="-0.001824 0.000 -0.052274" rpy="0 0 0"/>
+      <origin xyz="-0.001824 0 -0.052274" rpy="0 0 0"/>
       <mass value="0.029252"/>
-      <inertia ixx="0.000049199945" ixy="0.000" ixz="0.000000651855" iyy="0.000026577036" iyz="-0.000000219226" izz="0.000023937660"/>
+      <inertia ixx="0.000049199945" ixy="0" ixz="0.000000651855" iyy="0.000026577036" iyz="0" izz="0.000023937660"/>
     </inertial>
     <visual>
