Commit message: modify to use passive joint and enable walk

File: opr_description/robots/gankenkun_v4.xacro (robot description, xacro)
@@ -9,10 +9,10 @@
   <link name="base_link"/>
   <!-- uncomment this part to fixed the body in space (ignore gravity) -->
-  <!-- <link name="world"/>
-  <joint name="world2base" type="fixed">
-    <origin xyz="0 0 0" rpy="0 0 0"/>
-    <parent link="world"/>
-    <child link="base_link"/>
-  </joint> -->
+  <!--<link name="world"/>-->
+  <!--<joint name="world2base" type="fixed">-->
+  <!--  <origin xyz="0 0 0" rpy="0 0 0"/>-->
+  <!--  <parent link="world"/>-->
+  <!--  <child link="base_link"/>-->
+  <!--</joint>-->
   <!-- import robot parts -->
   <xacro:include filename="$(find opr_description)/urdf/version4/body/body.urdf.xacro"/>

File: opr_description/urdf/version4/arms/arms.gazebo.xacro (robot description, xacro)
@@ -3,11 +3,6 @@
   <xacro:macro name="arm_gazebo" params="name">
     <gazebo reference="${name}">
-      <mu1>1.0</mu1>
-      <mu2>1.0</mu2>
-      <kp>1000000.0</kp>
-      <kd>100.0</kd>
-      <gravity>false</gravity>
-      <minDepth>0.001</minDepth>
-      <maxVel>1.0</maxVel>
+      <mu1>0.2</mu1>
+      <mu2>0.0</mu2>
       <selfCollide>false</selfCollide>
     </gazebo>

File: opr_description/urdf/version4/arms/arms.transmission.xacro (robot description, xacro)
@@ -13,8 +13,8 @@
   </xacro:macro>
   <xacro:arm_transmission name="left_shoulder_pitch_joint"/>
-  <!-- <xacro:arm_transmission name="left_shoulder_roll_joint"/> -->
+  <xacro:arm_transmission name="left_shoulder_roll_joint"/>
   <xacro:arm_transmission name="left_elbow_pitch_joint"/>
   <xacro:arm_transmission name="right_shoulder_pitch_joint"/>
-  <!-- <xacro:arm_transmission name="right_shoulder_roll_joint"/> -->
+  <xacro:arm_transmission name="right_shoulder_roll_joint"/>
   <xacro:arm_transmission name="right_elbow_pitch_joint"/>
 </robot>

File: opr_description/urdf/version4/arms/left_arm.urdf.xacro (robot description, xacro)
@@ -8,4 +8,5 @@
     <limit effort="1000" lower="${-3*PI/4}" upper="${3*PI/4}" velocity="4.8"/>
     <axis xyz="0 1 0"/>
+    <dynamics damping="0.1" friction="0.0"/>
   </joint>
   <joint name="left_shoulder_roll_joint" type="revolute">
@@ -13,6 +14,7 @@
     <child link="left_arm_link"/>
     <origin xyz="0 0.03 0" rpy="0 0 0"/>
-    <limit effort="100" lower="0" upper="${PI}" velocity="4.8"/>
+    <limit effort="1000" lower="${-PI}" upper="${PI}" velocity="4.8"/>
     <axis xyz="1 0 0"/>
+    <dynamics damping="0.1" friction="0.0"/>
   </joint>
   <joint name="left_elbow_pitch_joint" type="revolute">
@@ -20,6 +22,7 @@
     <child link="left_forearm_link"/>
     <origin xyz="0 0 -0.109" rpy="0 0 0"/>
-    <limit effort="100" lower="${-3*PI/4}" upper="${3*PI/4}" velocity="4.8"/>
+    <limit effort="1000" lower="${-3*PI/4}" upper="${3*PI/4}" velocity="4.8"/>
     <axis xyz="0 1 0"/>
+    <dynamics damping="0.1" friction="0.0"/>
   </joint>
   <!-- arm links -->
@@ -47,5 +50,5 @@
       <origin xyz="-0.000173 -0.000173 -0.0545" rpy="0 0 0"/>
       <mass value="0.198342"/>
-      <inertia ixx="0.000398226787" ixy="0.000000017648" ixz="-0.000003440285" iyy="0.000398226787" iyz="0.000003440285" izz="0.000042097457"/>
+      <inertia ixx="0.000398226787" ixy="0.0" ixz="0.0" iyy="0.000398226787" iyz="0.0" izz="0.000042097457"/>
     </inertial>
     <visual>

File: opr_description/urdf/version4/arms/right_arm.urdf.xacro (robot description, xacro)
@@ -8,4 +8,5 @@
     <limit effort="1000" lower="${-3*PI/4}" upper="${3*PI/4}" velocity="4.8"/>
     <axis xyz="0 1 0"/>
+    <dynamics damping="0.1" friction="0.0"/>
   </joint>
   <joint name="right_shoulder_roll_joint" type="revolute">
@@ -13,6 +14,7 @@
     <child link="right_arm_link"/>
     <origin xyz="0 -0.03 0" rpy="0 0 0"/>
-    <limit effort="100" lower="${-PI}" upper="0" velocity="4.8"/>
+    <limit effort="1000" lower="${-PI}" upper="${PI}" velocity="4.8"/>
     <axis xyz="1 0 0"/>
+    <dynamics damping="0.1" friction="0.0"/>
   </joint>
   <joint name="right_elbow_pitch_joint" type="revolute">
@@ -20,6 +22,7 @@
     <child link="right_forearm_link"/>
     <origin xyz="0 0 -0.109" rpy="0 0 0"/>
-    <limit effort="100" lower="${-3*PI/4}" upper="${3*PI/4}" velocity="4.8"/>
+    <limit effort="1000" lower="${-3*PI/4}" upper="${3*PI/4}" velocity="4.8"/>
     <axis xyz="0 1 0"/>
+    <dynamics damping="0.1" friction="0.0"/>
   </joint>
   <!-- arm links -->
@@ -47,5 +50,6 @@
       <origin xyz="0.00049 -0.00049 -0.0545" rpy="0 0 0"/>
       <mass value="0.198342"/>
-      <inertia ixx="0.000398185104" ixy="0.000000071266" ixz="0.000000295835" iyy="0.000398185104" iyz="0.000000295835" izz="0.000042014091"/>
+      <!--<inertia ixx="0.000398185104" ixy="0.000000071266" ixz="0.000000295835" iyy="0.000398185104" iyz="0.000000295835" izz="0.000042014091"/>-->
+      <inertia ixx="0.000398185104" ixy="0.0" ixz="0.0" iyy="0.000398185104" iyz="0.0" izz="0.000042014091"/>
     </inertial>
     <visual>

File: opr_description/urdf/version4/body/body.gazebo.xacro (robot description, xacro)
@@ -2,12 +2,13 @@
 <robot xmlns:xacro="http://www.ros.org/wiki/xacro">
   <gazebo reference="body_link">
-    <mu1>1.0</mu1>
-    <mu2>1.0</mu2>
+    <mu1>0.01</mu1>
+    <mu2>0.0</mu2>
     <kp>1000000.0</kp>
     <kd>100.0</kd>
-    <gravity>false</gravity>
-    <minDepth>0.001</minDepth>
-    <maxVel>1.0</maxVel>
+    <maxVel>10.0</maxVel>
+    <minDepth>0.0001</minDepth>
+    <maxContacts>6</maxContacts>
     <selfCollide>false</selfCollide>
+    <dampingFactor>0</dampingFactor>
   </gazebo>
 </robot>

File: opr_description/urdf/version4/body/body.urdf.xacro (robot description, xacro)
@@ -11,5 +11,5 @@
     <inertial>
       <origin xyz="-0.022825 0.000073 -0.015720" rpy="0 0 0"/>
-      <mass value="1.645331"/>
+      <mass value="2.645331"/>
       <inertia ixx="0.007742297482" ixy="0.000005961013" ixz="0.000422502364" iyy="0.008034384246" iyz="-0.000003797186" izz="0.003984603997"/>
     </inertial>

File: opr_description/urdf/version4/head/head.gazebo.xacro (robot description, xacro)
@@ -2,11 +2,6 @@
 <robot xmlns:xacro="http://www.ros.org/wiki/xacro">
   <gazebo reference="head_yaw_link">
-    <mu1>1.0</mu1>
-    <mu2>1.0</mu2>
-    <kp>1000000.0</kp>
-    <kd>100.0</kd>
-    <gravity>false</gravity>
-    <minDepth>0.001</minDepth>
-    <maxVel>1.0</maxVel>
+    <mu1>0.2</mu1>
+    <mu2>0.0</mu2>
     <selfCollide>false</selfCollide>
   </gazebo>

File: opr_description/urdf/version4/head/head.urdf.xacro (robot description, xacro)
@@ -6,6 +6,7 @@
     <child link="head_yaw_link"/>
     <origin xyz="0 0 0.0875" rpy="0 0 0"/>
-    <limit effort="100" lower="${-3*PI/4}" upper="${3*PI/4}" velocity="4.8"/>
+    <limit effort="1000" lower="${-3*PI/4}" upper="${3*PI/4}" velocity="4.8"/>
     <axis xyz="0 0 1"/>
+    <dynamics damping="0.1" friction="0.0"/>
   </joint>
   <!-- head link -->

File: opr_description/urdf/version4/legs/left_leg.urdf.xacro (robot description, xacro)
@@ -8,4 +8,5 @@
     <limit effort="1000" lower="${-3*PI/4}" upper="${3*PI/4}" velocity="4.8"/>
     <axis xyz="0 0 1"/>
+    <dynamics damping="0.0" friction="0.0"/>
   </joint>
   <joint name="left_waist_roll_joint" type="revolute">
@@ -15,4 +16,5 @@
     <limit effort="1000" lower="${-PI/4}" upper="${PI/4}" velocity="4.8"/>
     <axis xyz="1 0 0"/>
+    <dynamics damping="0.1" friction="0.0"/>
   </joint>
   <joint name="left_waist_pitch_joint" type="revolute">
@@ -22,4 +24,5 @@
     <limit effort="1000" lower="${-PI/2}" upper="${PI/6}" velocity="4.8"/>
     <axis xyz="0 1 0"/>
+    <dynamics damping="0.1" friction="0.0"/>
   </joint>
   <joint name="left_knee_pitch_joint" type="revolute">
@@ -29,4 +32,5 @@
     <limit effort="1000" lower="${-PI/6}" upper="${PI/2}" velocity="4.8"/>
     <axis xyz="0 1 0"/>
+    <dynamics damping="0.1" friction="0.0"/>
   </joint>
   <joint name="left_ankle_pitch_joint" type="revolute">
@@ -36,4 +40,5 @@
     <limit effort="1000" lower="${-PI/2}" upper="${PI/2}" velocity="4.8"/>
     <axis xyz="0 1 0"/>
+    <dynamics damping="0.1" friction="0.0"/>
   </joint>
   <joint name="left_ankle_roll_joint" type="revolute">
@@ -43,4 +48,5 @@
     <limit effort="1000" lower="${-PI/2}" upper="${PI/2}" velocity="4.8"/>
     <axis xyz="1 0 0"/>
+    <dynamics damping="0.1" friction="0.0"/>
   </joint>
   <!-- mimic joints -->
@@ -51,5 +57,15 @@
     <limit effort="1000" lower="${-PI/2}" upper="${PI/2}" velocity="4.8"/>
     <axis xyz="1 0 0"/>
-    <mimic joint="left_waist_roll_joint" multiplier="-2" offset="0"/>
+    <mimic joint="left_waist_roll_joint" multiplier="2" offset="0"/>
+    <dynamics damping="0.0" friction="0.0"/>
+  </joint>
+  <joint name="left_knee_pitch_mimic_joint" type="revolute">
+    <parent link="left_thigh_link"/>
+    <child link="left_knee_link"/>
+    <origin xyz="0 0 -0.1" rpy="0 0 0"/>
+    <limit effort="1000" lower="${-PI/6}" upper="${PI/2}" velocity="4.8"/>
+    <axis xyz="0 1 0"/>
+    <mimic joint="left_waist_pitch_joint" multiplier="-1" offset="0"/>
+    <dynamics damping="0.1" friction="0.0"/>
   </joint>
   <joint name="left_hamstring_mimic_joint" type="revolute">
@@ -60,13 +76,5 @@
     <axis xyz="0 1 0"/>
     <mimic joint="left_waist_pitch_joint" multiplier="1" offset="0"/>
-  </joint>
-  <joint name="left_knee_pitch_mimic_joint" type="revolute">
-    <!-- closed loop -->
-    <parent link="left_thigh_link"/>
-    <child link="left_knee_link"/>
-    <origin xyz="0 0 -0.1" rpy="0 0 0"/>
-    <limit effort="1000" lower="${-PI/6}" upper="${PI/2}" velocity="4.8"/>
-    <axis xyz="0 1 0"/>
-    <mimic joint="left_waist_pitch_joint" multiplier="-1" offset="0"/>
+    <dynamics damping="0.1" friction="0.0"/>
   </joint>
   <joint name="left_calf_mimic_joint" type="revolute">
@@ -77,7 +85,7 @@
     <axis xyz="0 1 0"/>
     <mimic joint="left_knee_pitch_joint" multiplier="1" offset="0"/>
+    <dynamics damping="0.1" friction="0.0"/>
   </joint>
   <joint name="left_ankle_pitch_mimic_joint" type="revolute">
-    <!-- closed loop -->
     <parent link="left_shin_link"/>
     <child link="left_ankle_side_link"/>
@@ -86,4 +94,5 @@
     <axis xyz="0 1 0"/>
     <mimic joint="left_knee_pitch_joint" multiplier="-1" offset="0"/>
+    <dynamics damping="0.1" friction="0.0"/>
   </joint>
   <!-- leg links -->

File: opr_description/urdf/version4/legs/legs.gazebo.xacro (robot description, xacro)
@@ -12,47 +12,156 @@
     </gazebo>
   </xacro:macro>
-  <xacro:macro name="leg_gazebo" params="name">
+  <xacro:macro name="contact_disabled_link" params="name">
     <gazebo reference="${name}">
-      <mu1>1.0</mu1>
-      <mu2>1.0</mu2>
-      <kp>10000.0</kp>
-      <kd>100.0</kd>
-      <gravity>false</gravity>
-      <minDepth>0.001</minDepth>
-      <maxVel>1.0</maxVel>
+      <mu1>0</mu1>
+      <mu2>0</mu2>
+      <kp>10000000</kp>
+      <kd>0</kd>
       <selfCollide>false</selfCollide>
+      <collision>
+        <surface>
+          <contact>
+            <collide_without_contact>true</collide_without_contact>
+          </contact>
+        </surface>
+      </collision>
     </gazebo>
   </xacro:macro>
-  <xacro:leg_gazebo name="left_waist_yaw_link"/>
-  <xacro:leg_gazebo name="left_waist_roll_link"/>
-  <xacro:leg_gazebo name="left_thigh_link"/>
-  <xacro:leg_gazebo name="left_knee_link"/>
-  <xacro:leg_gazebo name="left_shin_link"/>
-  <xacro:leg_gazebo name="left_ankle_side_link"/>
-  <xacro:leg_gazebo name="left_ankle_link"/>
-  <xacro:leg_gazebo name="left_foot_link"/>
-  <xacro:leg_gazebo name="left_slider_crank_link"/>
-  <xacro:leg_gazebo name="left_hamstring_link"/>
-  <xacro:leg_gazebo name="left_calf_link"/>
-  <xacro:mimic_joint name="left_slider_crank_mimic_joint" parent="left_waist_roll_joint" multiplier="-2"/>
-  <xacro:mimic_joint name="left_hamstring_mimic_joint" parent="left_waist_pitch_joint" multiplier="1"/>
-  <xacro:mimic_joint name="left_knee_pitch_mimic_joint" parent="left_waist_pitch_joint" multiplier="-1"/>
-  <xacro:mimic_joint name="left_calf_mimic_joint" parent="left_knee_pitch_joint" multiplier="1"/>
-  <xacro:mimic_joint name="left_ankle_pitch_mimic_joint" parent="left_knee_pitch_joint" multiplier="-1"/>
-  <xacro:leg_gazebo name="right_waist_yaw_link"/>
-  <xacro:leg_gazebo name="right_waist_roll_link"/>
-  <xacro:leg_gazebo name="right_thigh_link"/>
-  <xacro:leg_gazebo name="right_knee_link"/>
-  <xacro:leg_gazebo name="right_shin_link"/>
-  <xacro:leg_gazebo name="right_ankle_side_link"/>
-  <xacro:leg_gazebo name="right_ankle_link"/>
-  <xacro:leg_gazebo name="right_foot_link"/>
-  <xacro:leg_gazebo name="right_slider_crank_link"/>
-  <xacro:leg_gazebo name="right_hamstring_link"/>
-  <xacro:leg_gazebo name="right_calf_link"/>
-  <xacro:mimic_joint name="right_slider_crank_mimic_joint" parent="right_waist_roll_joint" multiplier="-2"/>
-  <xacro:mimic_joint name="right_hamstring_mimic_joint" parent="right_waist_pitch_joint" multiplier="1"/>
-  <xacro:mimic_joint name="right_knee_pitch_mimic_joint" parent="right_waist_pitch_joint" multiplier="-1"/>
-  <xacro:mimic_joint name="right_calf_mimic_joint" parent="right_knee_pitch_joint" multiplier="1"/>
-  <xacro:mimic_joint name="right_ankle_pitch_mimic_joint" parent="right_knee_pitch_joint" multiplier="-1"/>
+  <xacro:macro name="leg_link" params="name">
+    <gazebo reference="${name}">
+      <mu1>0.2</mu1>
+      <mu2>0</mu2>
+      <kp>1000000.0</kp>
+      <kd>100.0</kd>
+      <maxVel>10.0</maxVel>
+      <minDepth>0.01</minDepth>
+      <maxContacts>6</maxContacts>
+      <selfCollide>false</selfCollide>
+      <dampingFactor>0</dampingFactor>
+    </gazebo>
+  </xacro:macro>
+  <xacro:macro name="foot_link" params="name">
+    <gazebo reference="${name}">
+      <!--<mu1>1.0</mu1>-->
+      <!--<mu2>0.0</mu2>-->
+      <!--<kp>1000000.0</kp>-->
+      <!--<kd>100.0</kd>-->
+      <!--<maxVel>10.0</maxVel>-->
+      <!--<minDepth>0.001</minDepth>-->
+      <!--<maxContacts>10</maxContacts>-->
+      <selfCollide>false</selfCollide>
+      <dampingFactor>0</dampingFactor>
+      <!--<mu1>100000</mu1>-->
+      <mu2>0.0</mu2>
+      <kp>1000000.0</kp>
+      <kd>10000.0</kd>
+      <maxVel>0.0</maxVel>
+      <minDepth>0.0</minDepth>
+      <maxContacts>6</maxContacts>
+      <!--<mu1>9000</mu1>-->
+      <!--<mu2>9000</mu2>-->
+      <!--<kp>1000000.0</kp>-->
+      <!--<kd>10.0</kd>-->
+      <!--<minDepth>0.001</minDepth>-->
+      <!--<maxContacts>10</maxContacts>-->
+    </gazebo>
+  </xacro:macro>
+  <xacro:macro name="implicit_joint" params="name">
+    <gazebo reference="${name}">
+      <physics>
+        <ode>
+          <implicit_spring_damper>1</implicit_spring_damper>
+        </ode>
+      </physics>
+    </gazebo>
+  </xacro:macro>
+  <xacro:macro name="passive_joint" params="name parent child xyz:='0 0 0' rpy:='0 0 0' axis:='0 1 0'">
+    <gazebo>
+      <joint name="${name}_passive_joint" type="revolute">
+        <parent>${parent}</parent>
+        <child>${child}</child>
+        <pose relative_to="${parent}">${xyz} ${rpy}</pose>
+        <axis>
+          <xyz>${axis}</xyz>
+          <limit>
+            <lower>-3.141</lower>
+            <upper>3.141</upper>
+            <effort>10000</effort>
+            <velocity>10000</velocity>
+          </limit>
+          <dynamics>
+            <damping>0</damping>
+            <friction>0</friction>
+            <spring_reference>0</spring_reference>
+            <spring_stiffness>0</spring_stiffness>
+          </dynamics>
+        </axis>
+        <physics>
+          <ode>
+            <implicit_spring_damper>1</implicit_spring_damper>
+          </ode>
+        </physics>
+      </joint>
+    </gazebo>
+  </xacro:macro>
+  <xacro:leg_link name="left_waist_yaw_link"/>
+  <xacro:leg_link name="left_waist_roll_link"/>
+  <xacro:leg_link name="left_thigh_link"/>
+  <xacro:leg_link name="left_knee_link"/>
+  <xacro:leg_link name="left_shin_link"/>
+  <xacro:leg_link name="left_ankle_side_link"/>
+  <xacro:leg_link name="left_ankle_link"/>
+  <xacro:foot_link name="left_foot_link"/>
+  <xacro:contact_disabled_link name="left_slider_crank_link"/>
+  <xacro:leg_link name="left_hamstring_link"/>
+  <xacro:leg_link name="left_calf_link"/>
+  <xacro:implicit_joint name="left_waist_yaw_joint"/>
+  <xacro:implicit_joint name="left_waist_roll_joint"/>
+  <xacro:implicit_joint name="left_slider_crank_mimic_joint"/>
+  <xacro:implicit_joint name="left_waist_pitch_joint"/>
+  <xacro:implicit_joint name="left_knee_pitch_mimic_joint"/>
+  <xacro:implicit_joint name="left_hamstring_mimic_joint"/>
+  <xacro:implicit_joint name="left_knee_pitch_joint"/>
+  <xacro:implicit_joint name="left_ankle_pitch_mimic_joint"/>
+  <xacro:implicit_joint name="left_calf_mimic_joint"/>
+  <xacro:implicit_joint name="left_ankle_pitch_joint"/>
+  <xacro:implicit_joint name="left_ankle_roll_joint"/>
+  <xacro:passive_joint name="left_slider_crank" parent="left_waist_yaw_link" child="left_slider_crank_link" xyz="-0.04 0 -0.0065" axis="1 0 0"/>
+  <xacro:passive_joint name="left_knee_pitch" parent="left_hamstring_link" child="left_knee_link" xyz="0 0 -0.1"/>
+  <xacro:passive_joint name="left_ankle_pitch" parent="left_calf_link" child="left_ankle_side_link" xyz="0 0 -0.1"/>
+  <!--<xacro:mimic_joint name="left_slider_crank_mimic_joint" parent="left_waist_roll_joint" multiplier="-2"/>-->
+  <!--<xacro:mimic_joint name="left_hamstring_mimic_joint" parent="left_waist_pitch_joint" multiplier="1"/>-->
+  <!--<xacro:mimic_joint name="left_knee_pitch_mimic_joint" parent="left_waist_pitch_joint" multiplier="-1"/>-->
+  <!--<xacro:mimic_joint name="left_calf_mimic_joint" parent="left_knee_pitch_joint" multiplier="1"/>-->
+  <!--<xacro:mimic_joint name="left_ankle_pitch_mimic_joint" parent="left_knee_pitch_joint" multiplier="-1"/>-->
+  <xacro:leg_link name="right_waist_yaw_link"/>
+  <xacro:leg_link name="right_waist_roll_link"/>
+  <xacro:leg_link name="right_thigh_link"/>
+  <xacro:leg_link name="right_knee_link"/>
+  <xacro:leg_link name="right_shin_link"/>
+  <xacro:leg_link name="right_ankle_side_link"/>
+  <xacro:leg_link name="right_ankle_link"/>
+  <xacro:foot_link name="right_foot_link"/>
+  <xacro:leg_link name="right_slider_crank_link"/>
+  <xacro:leg_link name="right_hamstring_link"/>
+  <xacro:leg_link name="right_calf_link"/>
+  <xacro:implicit_joint name="right_waist_yaw_joint"/>
+  <xacro:implicit_joint name="right_waist_roll_joint"/>
+  <xacro:implicit_joint name="right_slider_crank_mimic_joint"/>
+  <xacro:implicit_joint name="right_waist_pitch_joint"/>
+  <xacro:implicit_joint name="right_knee_pitch_mimic_joint"/>
+  <xacro:implicit_joint name="right_hamstring_mimic_joint"/>
+  <xacro:implicit_joint name="right_knee_pitch_joint"/>
+  <xacro:implicit_joint name="right_ankle_pitch_mimic_joint"/>
+  <xacro:implicit_joint name="right_calf_mimic_joint"/>
+  <xacro:implicit_joint name="right_ankle_pitch_joint"/>
+  <xacro:implicit_joint name="right_ankle_roll_joint"/>
+  <xacro:passive_joint name="right_slider_crank" parent="right_waist_yaw_link" child="right_slider_crank_link" xyz="-0.04 0 -0.0065" axis="1 0 0"/>
+  <xacro:passive_joint name="right_knee" parent="right_hamstring_link" child="right_knee_link" xyz="0 0 -0.1"/>
+  <xacro:passive_joint name="right_ankle" parent="right_calf_link" child="right_ankle_side_link" xyz="0 0 -0.1"/>
+  <!--<xacro:mimic_joint name="right_slider_crank_mimic_joint" parent="right_waist_roll_joint" multiplier="-2"/>-->
+  <!--<xacro:mimic_joint name="right_hamstring_mimic_joint" parent="right_waist_pitch_joint" multiplier="1"/>-->
+  <!--<xacro:mimic_joint name="right_knee_pitch_mimic_joint" parent="right_waist_pitch_joint" multiplier="-1"/>-->
+  <!--<xacro:mimic_joint name="right_calf_mimic_joint" parent="right_knee_pitch_joint" multiplier="1"/>-->
+  <!--<xacro:mimic_joint name="right_ankle_pitch_mimic_joint" parent="right_knee_pitch_joint" multiplier="-1"/>-->
 </robot>

File: opr_description/urdf/version4/legs/right_leg.urdf.xacro (robot description, xacro)
@@ -6,6 +6,7 @@
     <child link="right_waist_yaw_link"/>
     <origin xyz="0.004954 -0.044 -0.107" rpy="0 0 0"/>
-    <limit effort="100" lower="${-3*PI/4}" upper="${3*PI/4}" velocity="4.8"/>
+    <limit effort="1000" lower="${-3*PI/4}" upper="${3*PI/4}" velocity="4.8"/>
     <axis xyz="0 0 1"/>
+    <dynamics damping="0.1" friction="0.0"/>
   </joint>
   <joint name="right_waist_roll_joint" type="revolute">
@@ -15,4 +16,5 @@
     <limit effort="1000" lower="${-PI/4}" upper="${PI/4}" velocity="4.8"/>
     <axis xyz="1 0 0"/>
+    <dynamics damping="0.1" friction="0.0"/>
   </joint>
   <joint name="right_waist_pitch_joint" type="revolute">
@@ -22,4 +24,5 @@
     <limit effort="1000" lower="${-PI/2}" upper="${PI/6}" velocity="4.8"/>
     <axis xyz="0 1 0"/>
+    <dynamics damping="0.1" friction="0.0"/>
   </joint>
   <joint name="right_knee_pitch_joint" type="revolute">
@@ -29,4 +32,5 @@
     <limit effort="1000" lower="${-PI/6}" upper="${PI/2}" velocity="4.8"/>
     <axis xyz="0 1 0"/>
+    <dynamics damping="0.1" friction="0.0"/>
   </joint>
   <joint name="right_ankle_pitch_joint" type="revolute">
@@ -36,4 +40,5 @@
     <limit effort="1000" lower="${-PI/2}" upper="${PI/2}" velocity="4.8"/>
     <axis xyz="0 1 0"/>
+    <dynamics damping="0.1" friction="0.0"/>
   </joint>
   <joint name="right_ankle_roll_joint" type="revolute">
@@ -43,4 +48,5 @@
     <limit effort="1000" lower="${-PI/2}" upper="${PI/2}" velocity="4.8"/>
     <axis xyz="1 0 0"/>
+    <dynamics damping="0.1" friction="0.0"/>
   </joint>
   <!-- mimic joints -->
@@ -52,4 +58,5 @@
     <axis xyz="1 0 0"/>
     <mimic joint="right_waist_roll_joint" multiplier="-2" offset="0"/>
+    <dynamics damping="0.0" friction="0.0"/>
   </joint>
   <joint name="right_hamstring_mimic_joint" type="revolute">
@@ -60,7 +67,7 @@
     <axis xyz="0 1 0"/>
     <mimic joint="right_waist_pitch_joint" multiplier="1" offset="0"/>
+    <dynamics damping="0.1" friction="0.0"/>
   </joint>
   <joint name="right_knee_pitch_mimic_joint" type="revolute">
-    <!-- closed loop -->
     <parent link="right_thigh_link"/>
     <child link="right_knee_link"/>
@@ -69,4 +76,5 @@
     <axis xyz="0 1 0"/>
     <mimic joint="right_waist_pitch_joint" multiplier="-1" offset="0"/>
+    <dynamics damping="0.1" friction="0.0"/>
   </joint>
   <joint name="right_calf_mimic_joint" type="revolute">
@@ -77,7 +85,7 @@
     <axis xyz="0 1 0"/>
     <mimic joint="right_knee_pitch_joint" multiplier="1" offset="0"/>
+    <dynamics damping="0.1" friction="0.0"/>
   </joint>
   <joint name="right_ankle_pitch_mimic_joint" type="revolute">
-    <!-- closed loop -->
     <parent link="right_shin_link"/>
     <child link="right_ankle_side_link"/>
@@ -86,4 +94,5 @@
     <axis xyz="0 1 0"/>
     <mimic joint="right_knee_pitch_joint" multiplier="-1" offset="0"/>
+    <dynamics damping="0.1" friction="0.0"/>
   </joint>
   <!-- leg links -->
