Commit message: added imu

File: opr_description/robots/gankenkun_v4.xacro (robot description, xacro)
@@ -32,3 +32,8 @@
   <xacro:include filename="$(find opr_description)/urdf/version4/arms/arms.transmission.xacro"/>
   <xacro:include filename="$(find opr_description)/urdf/version4/legs/legs.transmission.xacro"/>
+  <!-- sensors -->
+  <xacro:include filename="$(find opr_description)/urdf/version4/sensors/imu/n100.xacro"/>
+  <xacro:n100_imu name="imu" parent="body_link" update_rate="100">
+    <origin xyz="0 0 0" rpy="0 0 0"/>
+  </xacro:n100_imu>
 </robot>

Commit message: added camera

File: opr_description/robots/gankenkun_v4.xacro (robot description, xacro)
@@ -37,3 +37,7 @@
     <origin xyz="0 0 0" rpy="0 0 0"/>
   </xacro:n100_imu>
+  <xacro:include filename="$(find opr_description)/urdf/version4/sensors/camera/camera.xacro"/>
+  <xacro:camera name="camera" parent="head_yaw_link">
+    <origin xyz="0.036496 0 0.055504" rpy="0 ${pi /4} 0"/>
+  </xacro:camera>
 </robot>

Commit message: move sensors

File: opr_description/robots/gankenkun_v4.xacro (robot description, xacro)
@@ -33,9 +33,9 @@
   <xacro:include filename="$(find opr_description)/urdf/version4/legs/legs.transmission.xacro"/>
   <!-- sensors -->
-  <xacro:include filename="$(find opr_description)/urdf/version4/sensors/imu/n100.xacro"/>
-  <xacro:n100_imu name="imu" parent="body_link" update_rate="100">
+  <xacro:include filename="$(find opr_description)/urdf/version4/sensors/imu.xacro"/>
+  <xacro:imu name="imu" parent="body_link" update_rate="100">
     <origin xyz="0 0 0" rpy="0 0 0"/>
-  </xacro:n100_imu>
-  <xacro:include filename="$(find opr_description)/urdf/version4/sensors/camera/camera.xacro"/>
+  </xacro:imu>
+  <xacro:include filename="$(find opr_description)/urdf/version4/sensors/camera.xacro"/>
   <xacro:camera name="camera" parent="head_yaw_link">
     <origin xyz="0.036496 0 0.055504" rpy="0 ${pi /4} 0"/>

File: opr_description/urdf/version4/sensors/imu.xacro (robot description, xacro)
@@ -1,6 +1,6 @@
 <?xml version="1.0" encoding="UTF-8"?>
 <robot xmlns:sensor="http://playerstage.sourceforge.net/gazebo/xmlschema/#sensor" xmlns:controller="http://playerstage.sourceforge.net/gazebo/xmlschema/#controller" xmlns:interface="http://playerstage.sourceforge.net/gazebo/xmlschema/#interface" xmlns:xacro="http://www.ros.org/wiki/xacro">
-  <xacro:include filename="n100_gazebo.xacro"/>
-  <xacro:macro name="n100_imu" params="name parent:='base_link' update_rate *origin">
+  <xacro:include filename="imu_gazebo.xacro"/>
+  <xacro:macro name="imu" params="name parent:='base_link' update_rate *origin">
     <xacro:property name="depth" value="0.05"/>
     <xacro:property name="width" value="0.05"/>
@@ -34,5 +34,5 @@
     </link>
     <!-- gazebo extensions -->
-    <xacro:n100_gazebo name="${name}" update_rate="${update_rate}"/>
+    <xacro:imu_gazebo name="${name}" update_rate="${update_rate}"/>
   </xacro:macro>
 </robot>

File: opr_description/urdf/version4/sensors/imu_gazebo.xacro (robot description, xacro)
@@ -1,5 +1,5 @@
 <?xml version="1.0" encoding="UTF-8"?>
 <robot xmlns:xacro="http://www.ros.org/wiki/xacro">
-  <xacro:macro name="n100_gazebo" params="name update_rate">
+  <xacro:macro name="imu_gazebo" params="name update_rate">
     <gazebo reference="${name}_link">
       <material>Gazebo/Gray</material>
